Commit message: fix: URDF and tools

File: urdf/minibot_middle_02.xacro (robot description, xacro)
@@ -23,9 +23,9 @@
     </visual>
   </link>
-  <xacro:property name="laser_d" value="0.06" />
-  <xacro:property name="laser_w" value="0.06" />
-  <xacro:property name="laser_h" value="0.06" />
+  <xacro:property name="laser_d" value="0.0386" />
+  <xacro:property name="laser_w" value="0.0386" />
+  <xacro:property name="laser_h" value="0.0339" />
   <xacro:property name="laser_x" value="0.0257" />
-  <xacro:property name="laser_z" value="0.0683" />
+  <xacro:property name="laser_z" value="0.0946" />
   <joint name="laser_joint" type="fixed">
     <origin xyz="${laser_x} 0 ${laser_z}" rpy="0 0 0"/>
